File: pcb/kicad/CBR_AdapterBoard/CBR_AdapterBoard.kicad_sch (KiCad schematic)
At the start: 7 parts, among them J1 2125201004, J2 2125201004, J3 2125201004, J4 2125201004, J5 2125201004, J6 2125201004, J7 Keihin_22_Pin

Commit message: - Interim checkin.
Other:
- note added: "6 x Molex Connectors (4 way - Mini Fit Jnr)"
- note added: "Jan 2026 - v0.2"
Changed lines of the file:
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@@
+    (effects (font (size 1.27 1.27)) (justify left bottom))
+  )
+  (text "6 x Molex Connectors (4 way - Mini Fit Jnr)" (at 92.456 21.971 0)
+    (effects (font (size 2.54 2.54)) (justify left bottom))
+  )
+  (text "Jan 2026 - v0.2" (at 210.439 194.183 0)
     (effects (font (size 1.27 1.27)) (justify left bottom))
   )

Commit message: - File corrections.
Parts:
- J1, J2, J3, J4, J5, J6: footprint AJK_MolexPin:4-Way-Molex_Connector-MiniFit-JNR -> Blackbird:4-Way-Molex_Connector-MiniFit-JNR
- J7: footprint AJK_MolexPin:AJK_Single_MolexPin_1.8mmHole -> Blackbird:Blackbird_22_pin_keihin
Changed lines of the file:
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@@
       (effects (font (size 1.524 1.524)) (justify left) hide)
     )
-    (property "Footprint" "AJK_MolexPin:4-Way-Molex_Connector-MiniFit-JNR" (id 2) (at 169.037 28.067 0)
+    (property "Footprint" "Blackbird:4-Way-Molex_Connector-MiniFit-JNR" (id 2) (at 169.037 28.067 0)
       (effects (font (size 1.27 1.27) italic) hide)
     )
-    (property "Datasheet" "https://www.molex.com/en-us/products/part-detail-pdf/2125201004?display=pdf" (id 3) (at 169.037 28.067 0)
+    (property "Datasheet" "" (id 3) (at 169.037 28.067 0)
       (effects (font (size 1.27 1.27) italic) hide)
     )
@@
       (effects (font (size 1.524 1.524)) (justify left) hide)
     )
-    (property "Footprint" "AJK_MolexPin:4-Way-Molex_Connector-MiniFit-JNR" (id 2) (at 126.238 28.702 0)
+    (property "Footprint" "Blackbird:4-Way-Molex_Connector-MiniFit-JNR" (id 2) (at 126.238 28.702 0)
       (effects (font (size 1.27 1.27) italic) hide)
     )
-    (property "Datasheet" "https://www.molex.com/en-us/products/part-detail-pdf/2125201004?display=pdf" (id 3) (at 126.238 28.702 0)
+    (property "Datasheet" "" (id 3) (at 126.238 28.702 0)
       (effects (font (size 1.27 1.27) italic) hide)
     )
@@
       (effects (font (size 1.524 1.524)) (justify left) hide)
     )
-    (property "Footprint" "AJK_MolexPin:4-Way-Molex_Connector-MiniFit-JNR" (id 2) (at 81.788 28.702 0)
+    (property "Footprint" "Blackbird:4-Way-Molex_Connector-MiniFit-JNR" (id 2) (at 81.788 28.702 0)
       (effects (font (size 1.27 1.27) italic) hide)
     )
-    (property "Datasheet" "https://www.molex.com/en-us/products/part-detail-pdf/2125201004?display=pdf" (id 3) (at 81.788 28.702 0)
+    (property "Datasheet" "" (id 3) (at 81.788 28.702 0)
       (effects (font (size 1.27 1.27) italic) hide)
     )
@@
       (effects (font (size 1.524 1.524)) (justify left))
     )
-    (property "Footprint" "AJK_MolexPin:AJK_Single_MolexPin_1.8mmHole" (id 2) (at 140.97 143.51 0)
+    (property "Footprint" "Blackbird:Blackbird_22_pin_keihin" (id 2) (at 140.97 143.51 0)
       (effects (font (size 1.27 1.27) italic) hide)
     )
@@
     (pin "9")
   )
-  (symbol (lib_id "AJK_Molex-Way:2125201004") (at 38.481 28.702 0) (unit 1)
+  (symbol (lib_name "2125201004_1") (lib_id "AJK_Molex-Way:2125201004") (at 38.481 28.702 0) (unit 1)
     (in_bom yes) (on_board yes) (fields_autoplaced)
     (property "Reference" "J1" (id 0) (at 52.324 31.242 0)
@@
       (effects (font (size 1.524 1.524)) (justify left) hide)
     )
-    (property "Footprint" "AJK_MolexPin:4-Way-Molex_Connector-MiniFit-JNR" (id 2) (at 38.481 28.702 0)
+    (property "Footprint" "Blackbird:4-Way-Molex_Connector-MiniFit-JNR" (id 2) (at 38.481 28.702 0)
       (effects (font (size 1.27 1.27) italic) hide)
     )
@@
       (effects (font (size 1.524 1.524)) (justify left) hide)
     )
-    (property "Footprint" "AJK_MolexPin:4-Way-Molex_Connector-MiniFit-JNR" (id 2) (at 212.09 29.21 0)
+    (property "Footprint" "Blackbird:4-Way-Molex_Connector-MiniFit-JNR" (id 2) (at 212.09 29.21 0)
       (effects (font (size 1.27 1.27) italic) hide)
     )
-    (property "Datasheet" "https://www.molex.com/en-us/products/part-detail-pdf/2125201004?display=pdf" (id 3) (at 212.09 29.21 0)
+    (property "Datasheet" "" (id 3) (at 212.09 29.21 0)
       (effects (font (size 1.27 1.27) italic) hide)
     )
@@
       (effects (font (size 1.524 1.524)) (justify left) hide)
     )
-    (property "Footprint" "AJK_MolexPin:4-Way-Molex_Connector-MiniFit-JNR" (id 2) (at 252.984 28.956 0)
+    (property "Footprint" "Blackbird:4-Way-Molex_Connector-MiniFit-JNR" (id 2) (at 252.984 28.956 0)
       (effects (font (size 1.27 1.27) italic) hide)
     )
-    (property "Datasheet" "https://www.molex.com/en-us/products/part-detail-pdf/2125201004?display=pdf" (id 3) (at 252.984 28.956 0)
+    (property "Datasheet" "" (id 3) (at 252.984 28.956 0)
       (effects (font (size 1.27 1.27) italic) hide)
     )
@@
   (symbol_instances
     (path "/c42603fc-6669-4866-b876-8c78cb514c78"
-      (reference "J1") (unit 1) (value "2125201004") (footprint "AJK_MolexPin:4-Way-Molex_Connector-MiniFit-JNR")
+      (reference "J1") (unit 1) (value "2125201004") (footprint "Blackbird:4-Way-Molex_Connector-MiniFit-JNR")
     )
     (path "/997523c6-7449-409b-b7d6-13e4e8882e25"
-      (reference "J2") (unit 1) (value "2125201004") (footprint "AJK_MolexPin:4-Way-Molex_Connector-MiniFit-JNR")
+      (reference "J2") (unit 1) (value "2125201004") (footprint "Blackbird:4-Way-Molex_Connector-MiniFit-JNR")
     )
     (path "/795b6a9d-fae6-4156-b2f8-51dea025b863"
-      (reference "J3") (unit 1) (value "2125201004") (footprint "AJK_MolexPin:4-Way-Molex_Connector-MiniFit-JNR")
+      (reference "J3") (unit 1) (value "2125201004") (footprint "Blackbird:4-Way-Molex_Connector-MiniFit-JNR")
     )
     (path "/3d8543c5-66c1-42cd-9535-753e885dcb73"
-      (reference "J4") (unit 1) (value "2125201004") (footprint "AJK_MolexPin:4-Way-Molex_Connector-MiniFit-JNR")
+      (reference "J4") (unit 1) (value "2125201004") (footprint "Blackbird:4-Way-Molex_Connector-MiniFit-JNR")
     )
     (path "/c723bbb4-c03d-4faa-80a7-5048bd0cd28d"
-      (reference "J5") (unit 1) (value "2125201004") (footprint "AJK_MolexPin:4-Way-Molex_Connector-MiniFit-JNR")
+      (reference "J5") (unit 1) (value "2125201004") (footprint "Blackbird:4-Way-Molex_Connector-MiniFit-JNR")
     )
     (path "/e24b9aba-9cc9-4e59-ba41-7a1ac9106177"
-      (reference "J6") (unit 1) (value "2125201004") (footprint "AJK_MolexPin:4-Way-Molex_Connector-MiniFit-JNR")
+      (reference "J6") (unit 1) (value "2125201004") (footprint "Blackbird:4-Way-Molex_Connector-MiniFit-JNR")
     )
     (path "/a4784c3b-c2b6-4112-9818-881a29bf33ec"
-      (reference "J7") (unit 1) (value "Keihin_22_Pin") (footprint "AJK_MolexPin:AJK_Single_MolexPin_1.8mmHole")
+      (reference "J7") (unit 1) (value "Keihin_22_Pin") (footprint "Blackbird:Blackbird_22_pin_keihin")
     )
   )

Commit message: - File corrections.
Parts:
- J7: symbol AJK_SingleMolexPin:AJK_Molex_22_Pin -> Blackbird:Blackbird_Keihin_22_Pin
Changed lines of the file:
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@@
     (pin "4")
   )
-  (symbol (lib_id "AJK_SingleMolexPin:AJK_Molex_22_Pin") (at 144.78 101.6 0) (unit 1)
+  (symbol (lib_id "Blackbird:Blackbird_Keihin_22_Pin") (at 144.78 101.6 0) (unit 1)
     (in_bom yes) (on_board yes)
     (property "Reference" "J7" (id 0) (at 122.301 101.6 0)
@@
       (effects (font (size 1.524 1.524)) (justify left))
     )
-    (property "Footprint" "Blackbird:Blackbird_22_pin_keihin" (id 2) (at 140.97 143.51 0)
+    (property "Footprint" "Blackbird:Blackbird_22_pin_keihin" (id 2) (at 135.89 133.35 0)
       (effects (font (size 1.27 1.27) italic) hide)
     )
-    (property "Datasheet" "" (id 3) (at 151.13 147.32 0)
+    (property "Datasheet" "" (id 3) (at 146.05 137.16 0)
       (effects (font (size 1.27 1.27) italic) hide)
     )

Commit message: - File corrections.
Parts:
- J1, J2, J3, J4, J5, J6: symbol AJK_Molex-Way:2125201004 -> Blackbird:Molex-4-Way
Changed lines of the file:
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@@
     )
   )
-  (symbol (lib_id "AJK_Molex-Way:2125201004") (at 169.037 28.067 0) (unit 1)
+  (symbol (lib_name "Molex-4-Way_4") (lib_id "Blackbird:Molex-4-Way") (at 169.037 28.067 0) (unit 1)
     (in_bom yes) (on_board yes) (fields_autoplaced)
     (property "Reference" "J4" (id 0) (at 183.261 30.607 0)
@@
       (effects (font (size 1.27 1.27) italic) hide)
     )
-    (property "Datasheet" "" (id 3) (at 169.037 28.067 0)
+    (property "Datasheet" "https://www.molex.com/en-us/products/part-detail-pdf/Molex-4-Way?display=pdf" (id 3) (at 169.037 28.067 0)
       (effects (font (size 1.27 1.27) italic) hide)
     )
@@
     (pin "4")
   )
-  (symbol (lib_id "AJK_Molex-Way:2125201004") (at 126.238 28.702 0) (unit 1)
+  (symbol (lib_name "Molex-4-Way_3") (lib_id "Blackbird:Molex-4-Way") (at 126.238 28.702 0) (unit 1)
     (in_bom yes) (on_board yes) (fields_autoplaced)
     (property "Reference" "J3" (id 0) (at 140.462 31.242 0)
@@
       (effects (font (size 1.27 1.27) italic) hide)
     )
-    (property "Datasheet" "" (id 3) (at 126.238 28.702 0)
+    (property "Datasheet" "https://www.molex.com/en-us/products/part-detail-pdf/Molex-4-Way?display=pdf" (id 3) (at 126.238 28.702 0)
       (effects (font (size 1.27 1.27) italic) hide)
     )
@@
     (pin "4")
   )
-  (symbol (lib_id "AJK_Molex-Way:2125201004") (at 81.788 28.702 0) (unit 1)
+  (symbol (lib_name "Molex-4-Way_2") (lib_id "Blackbird:Molex-4-Way") (at 81.788 28.702 0) (unit 1)
     (in_bom yes) (on_board yes)
     (property "Reference" "J2" (id 0) (at 96.012 31.242 0)
@@
       (effects (font (size 1.27 1.27) italic) hide)
     )
-    (property "Datasheet" "" (id 3) (at 81.788 28.702 0)
+    (property "Datasheet" "https://www.molex.com/en-us/products/part-detail-pdf/Molex-4-Way?display=pdf" (id 3) (at 81.788 28.702 0)
       (effects (font (size 1.27 1.27) italic) hide)
     )
@@
     (pin "9")
   )
-  (symbol (lib_name "2125201004_1") (lib_id "AJK_Molex-Way:2125201004") (at 38.481 28.702 0) (unit 1)
+  (symbol (lib_name "Molex-4-Way_1") (lib_id "Blackbird:Molex-4-Way") (at 38.481 28.702 0) (unit 1)
     (in_bom yes) (on_board yes) (fields_autoplaced)
     (property "Reference" "J1" (id 0) (at 52.324 31.242 0)
@@
     (pin "4")
   )
-  (symbol (lib_id "AJK_Molex-Way:2125201004") (at 212.09 29.21 0) (unit 1)
+  (symbol (lib_name "Molex-4-Way_5") (lib_id "Blackbird:Molex-4-Way") (at 212.09 29.21 0) (unit 1)
     (in_bom yes) (on_board yes) (fields_autoplaced)
     (property "Reference" "J5" (id 0) (at 226.314 31.75 0)
@@
       (effects (font (size 1.27 1.27) italic) hide)
     )
-    (property "Datasheet" "" (id 3) (at 212.09 29.21 0)
+    (property "Datasheet" "https://www.molex.com/en-us/products/part-detail-pdf/Molex-4-Way?display=pdf" (id 3) (at 212.09 29.21 0)
       (effects (font (size 1.27 1.27) italic) hide)
     )
@@
     (pin "4")
   )
-  (symbol (lib_id "AJK_Molex-Way:2125201004") (at 252.984 28.956 0) (unit 1)
+  (symbol (lib_id "Blackbird:Molex-4-Way") (at 252.984 28.956 0) (unit 1)
     (in_bom yes) (on_board yes) (fields_autoplaced)
     (property "Reference" "J6" (id 0) (at 267.208 31.496 0)
@@
       (effects (font (size 1.27 1.27) italic) hide)
     )
-    (property "Datasheet" "" (id 3) (at 252.984 28.956 0)
+    (property "Datasheet" "https://www.molex.com/en-us/products/part-detail-pdf/Molex-4-Way?display=pdf" (id 3) (at 252.984 28.956 0)
       (effects (font (size 1.27 1.27) italic) hide)
     )
